Commit message: updated tray

File: gym_blg/envs/data/tray/tray_old.urdf (robot description, URDF)
Before this commit: robot tray, 1 links, 0 joints
Links:
- link tray_base_link: mass 1 -> 0; geometry collision mesh filename=tray_textured.obj scale=0.5 0.5 0.5; visual mesh filename=tray_textured.obj scale=0.5 0.5 0.5
